File: SapphireMini_DLHR.sch (KiCad schematic (older format))
At the start: 15 parts, among them IC301 DLHR-F50D-E1BD-C-NAV8, U301 LIS331DLHTR

Commit message: From RA_Old Modified"
Parts:
- added C? (x2): 100nF, Capacitor_SMD:C_0603_1608Metric, symbol Device:C_Small
- added R? (x2): 47, Resistor_SMD:R_0603_1608Metric, symbol Device:R_Small_US
- added R? (x2): 4K75, Resistor_SMD:R_0603_1608Metric, symbol Device:R_Small_US
- added U?: BMP388, PQFN50P200X200X80-10N, symbol BMP388:BMP388
Connections:
- net labels added: ACC_INT1, ACC_INT2, BMP_INT
- wire segments 88 -> 114
- no-connect marks 3 -> 2
Other:
- moved on the sheet: C304, C305, R303, R304, R305, R306, R307, U301
