File: SapphireMini_Proc.sch (KiCad schematic (older format))
At the start: 66 parts, among them J501 Conn_02x05_Odd_Even, J502 Conn_01x03_Male, J503 USB_B_Micro, J504 Conn_01x05_Male, J505 Conn_01x08_Female, J506 Conn_01x08_Female, J507 Conn_01x04_Male, SW501 EVQP7C01P, U501 ATSAMD21E18A-AUT, U502 BMP388, U503 MB85RS1MT

Commit message: From RA_Old Modified"
Parts:
- removed C506, C507: 100nF, Capacitor_SMD:C_0603_1608Metric, symbol Device:C_Small
- removed R529, R530: 4K75, Resistor_SMD:R_0603_1608Metric, symbol Device:R_Small_US
- removed U502: BMP388, PQFN50P200X200X80-10N, symbol BMP388:BMP388
Connections:
- wire segments 299 -> 276
- no-connect marks 10 -> 9
Changed lines of the file:
@@
 $Descr USLetter 11000 8500
 encoding utf-8
-Sheet 5 7
+Sheet 6 8
 Title "Sapphire Mini"
 Date ""
@@
 Wire Wire Line
 	5850 1700 5850 1750
-Text Label 9700 950  0    50   ~ 0
-P3V3
-Wire Wire Line
-	9400 1050 9850 1050
-$Comp
-L Device:C_Small C506
-U 1 1 5FBCCD7A
-P 9850 1200
-F 0 "C506" H 9942 1246 50  0000 L CNN
-F 1 "100nF" H 9942 1155 50  0000 L CNN
-F 2 "Capacitor_SMD:C_0603_1608Metric" H 9850 1200 50  0001 C CNN
-F 3 "~" H 9850 1200 50  0001 C CNN
-F 4 "0.10" H 9850 1200 50  0001 C CNN "DigiKey Price"
-F 5 "CL10B104KA8NNNC" H 9850 1200 50  0001 C CNN "MPN"
-F 6 "Samsung" H 9850 1200 50  0001 C CNN "Manufacturer"
-F 7 "10%" H 9850 1200 50  0001 C CNN "Tolerance"
-F 8 "25" H 9850 1200 50  0001 C CNN "Voltage"
-F 9 "25 volt" H 9850 1200 50  0001 C CNN "Voltage Rating (DC)"
-F 10 "1" H 9850 1200 50  0001 C CNN "Populate"
-F 11 "MF-CAP-0603-0.1uF" H 9850 1200 50  0001 C CNN "MacroFab_PN"
-F 12 "1276-1006-1-ND " H 9850 1200 50  0001 C CNN "Digi-Key_PN"
-F 13 "Digikey" H 9850 1200 50  0001 C CNN "Distributor"
-F 14 "1276-1006-1-ND " H 9850 1200 50  0001 C CNN "DPN"
-F 15 "0.1 µF ±10% 25V Ceramic Capacitor X7R 0603 (1608 Metric)" H 9850 1200 50  0001 C CNN "Description"
-	1    9850 1200
-	1    0    0    -1
-$EndComp
-Wire Wire Line
-	9850 1100 9850 1050
-Connection ~ 9850 1050
-Wire Wire Line
-	9850 1050 9950 1050
-$Comp
-L Device:C_Small C507
-U 1 1 5FBDA68C
-P 10150 1100
-F 0 "C507" H 10242 1146 50  0000 L CNN
-F 1 "100nF" H 10242 1055 50  0000 L CNN
-F 2 "Capacitor_SMD:C_0603_1608Metric" H 10150 1100 50  0001 C CNN
-F 3 "~" H 10150 1100 50  0001 C CNN
-F 4 "0.10" H 10150 1100 50  0001 C CNN "DigiKey Price"
-F 5 "CL10B104KA8NNNC" H 10150 1100 50  0001 C CNN "MPN"
-F 6 "Samsung" H 10150 1100 50  0001 C CNN "Manufacturer"
-F 7 "10%" H 10150 1100 50  0001 C CNN "Tolerance"
-F 8 "25" H 10150 1100 50  0001 C CNN "Voltage"
-F 9 "25 volt" H 10150 1100 50  0001 C CNN "Voltage Rating (DC)"
-F 10 "1" H 10150 1100 50  0001 C CNN "Populate"
-F 11 "MF-CAP-0603-0.1uF" H 10150 1100 50  0001 C CNN "MacroFab_PN"
-F 12 "1276-1006-1-ND " H 10150 1100 50  0001 C CNN "Digi-Key_PN"
-F 13 "Digikey" H 10150 1100 50  0001 C CNN "Distributor"
-F 14 "1276-1006-1-ND " H 10150 1100 50  0001 C CNN "DPN"
-F 15 "0.1 µF ±10% 25V Ceramic Capacitor X7R 0603 (1608 Metric)" H 10150 1100 50  0001 C CNN "Description"
-	1    10150 1100
-	1    0    0    -1
-$EndComp
-Wire Wire Line
-	9400 950  10150 950
-Wire Wire Line
-	10150 1000 10150 950
-Connection ~ 10150 950
-Wire Wire Line
-	10150 950  10350 950
-Text Label 9700 1050 0    50   ~ 0
-P3V3
-$Comp
-L power:GND #PWR01
-U 1 1 5FBF3E4D
-P 9450 1900
-F 0 "#PWR01" H 9450 1650 50  0001 C CNN
-F 1 "GND" H 9455 1727 50  0000 C CNN
-F 2 "" H 9450 1900 50  0001 C CNN
-F 3 "" H 9450 1900 50  0001 C CNN
-	1    9450 1900
-	1    0    0    -1
-$EndComp
-$Comp
-L power:GND #PWR02
-U 1 1 5FBF4398
-P 9850 1300
-F 0 "#PWR02" H 9850 1050 50  0001 C CNN
-F 1 "GND" H 9855 1127 50  0000 C CNN
-F 2 "" H 9850 1300 50  0001 C CNN
-F 3 "" H 9850 1300 50  0001 C CNN
-	1    9850 1300
-	1    0    0    -1
-$EndComp
-$Comp
-L power:GND #PWR03
-U 1 1 5FBF477C
-P 10150 1200
-F 0 "#PWR03" H 10150 950 50  0001 C CNN
-F 1 "GND" H 10155 1027 50  0000 C CNN
-F 2 "" H 10150 1200 50  0001 C CNN
-F 3 "" H 10150 1200 50  0001 C CNN
-	1    10150 1200
-	1    0    0    -1
-$EndComp
-Wire Wire Line
-	9400 1850 9450 1900
-Wire Wire Line
-	8400 1350 8150 1350
-Text Label 8100 1350 0    50   ~ 0
-I2C_SCL
-Text Label 8100 1550 0    50   ~ 0
-I2C_SDA
-$Comp
-L Device:R_Small_US R530
-U 1 1 5FC1AA99
-P 8150 950
-F 0 "R530" H 8000 1050 50  0000 L CNN
-F 1 "4K75" H 7900 950 50  0000 L CNN
-F 2 "Resistor_SMD:R_0603_1608Metric" H 8150 950 50  0001 C CNN
-F 3 "~" H 8150 950 50  0001 C CNN
-F 4 "0.05" H 8150 950 50  0001 C CNN "DigiKey Price"
-F 5 "Vishay" H 8150 950 50  0001 C CNN "Manufacturer"
-F 6 "CRCW06034K75FKEAC" H 8150 950 50  0001 C CNN "MPN"
-F 7 "5%" H 8150 950 50  0001 C CNN "Tolerance"
-F 8 "1" H 8150 950 50  0001 C CNN "Populate"
-F 9 "CRCW060347K5FKEAC" H 8150 950 50  0001 C CNN "MacroFab_PN"
-F 10 "541-3984-1-ND" H 8150 950 50  0001 C CNN "Digi-Key_PN"
-F 11 "Digikey" H 8150 950 50  0001 C CNN "Distributor"
-F 12 "541-3984-1-ND " H 8150 950 50  0001 C CNN "DPN"
-F 13 "4.75 kOhms ±1% 0.1W, 1/10W Chip Resistor 0603" H 8150 950 50  0001 C CNN "Description"
-	1    8150 950
-	1    0    0    -1
-$EndComp
-$Comp
-L Device:R_Small_US R529
-U 1 1 5FC1B8CE
-P 7950 1100
-F 0 "R529" H 7800 1150 50  0000 L CNN
-F 1 "4K75" H 7700 1050 50  0000 L CNN
-F 2 "Resistor_SMD:R_0603_1608Metric" H 7950 1100 50  0001 C CNN
-F 3 "~" H 7950 1100 50  0001 C CNN
-F 4 "0.05" H 7950 1100 50  0001 C CNN "DigiKey Price"
-F 5 "Vishay" H 7950 1100 50  0001 C CNN "Manufacturer"
-F 6 "CRCW06034K75FKEAC" H 7950 1100 50  0001 C CNN "MPN"
-F 7 "5%" H 7950 1100 50  0001 C CNN "Tolerance"
-F 8 "1" H 7950 1100 50  0001 C CNN "Populate"
-F 9 "CRCW060347K5FKEAC" H 7950 1100 50  0001 C CNN "MacroFab_PN"
-F 10 "541-3984-1-ND" H 7950 1100 50  0001 C CNN "Digi-Key_PN"
-F 11 "Digikey" H 7950 1100 50  0001 C CNN "Distributor"
-F 12 "541-3984-1-ND " H 7950 1100 50  0001 C CNN "DPN"
-F 13 "4.75 kOhms ±1% 0.1W, 1/10W Chip Resistor 0603" H 7950 1100 50  0001 C CNN "Description"
-	1    7950 1100
-	1    0    0    -1
-$EndComp
-Wire Wire Line
-	8150 1050 8150 1350
-Wire Wire Line
-	8150 1350 8050 1350
-Connection ~ 8150 1350
-Wire Wire Line
-	7950 1550 7950 1200
-Wire Wire Line
-	7950 1550 8400 1550
-Wire Wire Line
-	7850 1550 7950 1550
-Connection ~ 7950 1550
-Wire Wire Line
-	8150 850  8150 650
-Wire Wire Line
-	7950 1000 7950 650
-Wire Wire Line
-	7700 650  7950 650
-Connection ~ 7950 650
-Wire Wire Line
-	7950 650  8150 650
-Connection ~ 8150 650
-Wire Wire Line
-	8150 650  8250 650
-Text Label 7950 650  0    50   ~ 0
-P3V3
-NoConn ~ 8400 1250
 NoConn ~ 4400 -450
 $Comp
@@
 Text Label 8750 2750 0    50   ~ 0
 I2C_SCL
-$Comp
-L power:GND #PWR0108
-U 1 1 5FB974AE
-P 8200 1900
-F 0 "#PWR0108" H 8200 1650 50  0001 C CNN
-F 1 "GND" H 8205 1727 50  0000 C CNN
-F 2 "" H 8200 1900 50  0001 C CNN
-F 3 "" H 8200 1900 50  0001 C CNN
-	1    8200 1900
-	1    0    0    -1
-$EndComp
-Wire Wire Line
-	8400 1650 8250 1650
-Wire Wire Line
-	8250 1650 8200 1700
-Wire Wire Line
-	8200 1700 8200 1900
 Text Label 6950 1700 0    50   ~ 0
-BMP_INT
-Wire Wire Line
-	9400 1250 9400 1650
-Wire Wire Line
-	9400 1650 10100 1650
-Text Label 9650 1650 0    50   ~ 0
 BMP_INT
 Text Label 1000 7850 0    50   ~ 0
@@
 Wire Wire Line
 	5550 4050 5700 4050
-$Comp
-L BMP388:BMP388 U502
-U 1 1 5FB8A4C9
-P 8900 1450
-F 0 "U502" H 8900 2217 50  0000 C CNN
-F 1 "BMP388" H 8900 2126 50  0000 C CNN
-F 2 "PQFN50P200X200X80-10N" H 8900 1450 50  0001 L BNN
-F 3 "" H 8900 1450 50  0001 L BNN
-F 4 "1.1" H 8900 1450 50  0001 L BNN "PARTREV"
-F 5 "IPC 7351B" H 8900 1450 50  0001 L BNN "STANDARD"
-F 6 "" H 8900 1450 50  0001 L BNN "MANUFACTURER"
-F 7 "828-1079-1-ND" H 8900 1450 50  0001 C CNN "DPN"
-F 8 "BMP388" H 8900 1450 50  0001 C CNN "MPN"
-F 9 "Bosch" H 8900 1450 50  0001 C CNN "Manufacturer"
-F 10 "1" H 8900 1450 50  0001 C CNN "Populate"
-F 11 "Pressure Sensor 4.35PSI ~ 18.13PSI (30kPa ~ 125kPa) Absolute - - 10-WFLGA" H 8900 1450 50  0001 C CNN "Description"
-F 12 "828-1079-1-ND " H 8900 1450 50  0001 C CNN "Digi-Key_PN"
-F 13 "120" H 8900 1450 50  0001 C CNN "OnHand"
-F 14 "MiniReel" H 8900 1450 50  0001 C CNN "Status"
-F 15 "Digikey" H 8900 1450 50  0001 C CNN "Distributor"
-	1    8900 1450
-	1    0    0    -1
-$EndComp
 Text Label 9350 3550 0    50   ~ 0
 VBAT_EN
@@
 Wire Wire Line
 	4000 7000 4900 7000
+Text HLabel 1800 -100 0    50   Input ~ 0
+P3V3
 $EndSCHEMATC
