File: SapphireMini_Pwr.sch (KiCad schematic (older format))
At the start: 27 parts, among them J201 JST, Q201 BC857BS, Q202 IRLML6402TRPBF, U201 TPS62150, U202 INA219BIDR

Commit message: From RA_Old Modified"
Parts:
- removed C204: 100nF, Capacitor_SMD:C_0603_1608Metric, symbol Device:C_Small
- removed C207: 1uF, Capacitor_SMD:C_0805_2012Metric, symbol Device:C_Small
- removed R209, R210: 10K, Resistor_SMD:R_0603_1608Metric, symbol Device:R_Small_US
- removed R211, R212: 10, Resistor_SMD:R_0603_1608Metric, symbol Device:R_Small_US
- removed U202: INA219BIDR, Package_SO:SOIC-8_3.9x4.9mm_P1.27mm, symbol Analog_ADC:INA219AxD
- R208: value 0.1 -> 0; MPN WSL0603R1000FEA -> (none)
Connections:
- net VBAT: now also Q201.4 (E2), Q202.3 (D), S201.1, S201.5; no longer J201.1 (Pin_1), S201.2, S201.6
- new net: J201.1 (Pin_1), S201.2, S201.6
Other:
- note added: "Current monitoring resistor if needed"
- note removed: "Revision 9: R211 and R212 \nchanged from 100K to 10 ohms \nto handle problems with bias offset\nand moved R208 (0.1 ohm current sense)\nto PWR IN line rather than P3V3"
