File: SapphireMini_DLHR.kicad_sch (KiCad schematic)
At the start: 17 parts, among them IC201 DLHR-F50D-E1BD-C-NAV8, U201 LIS331DLHTR, U202 BMP390, U203 MS5525DSO

Commit message: Start of layout
Parts:
- C201: footprint Capacitor_SMD:C_1206_3216Metric -> Capacitor_SMD:C_0805_2012Metric
- C202, C203, C204, C205, C207: footprint Capacitor_SMD:C_0603_1608Metric -> Capacitor_SMD:C_0402_1005Metric
- R201: MPN (none) -> EXB-2HV470JV
- U201: MPN (none) -> LIS331DLHTR
- U203: footprint SapphineMinimal:TE_MS5525DSO-DBxxxyS -> Sapphire:TE_5525DSO-DB001DS; MPN (none) -> 5525DSO-DB001DS
Connections:
- net GND: now also U203.9 (SUPPLY-)
- no-connect marks 4 -> 5
Changed lines of the file:
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@@
   (junction (at 198.12 149.86) (diameter 0) (color 0 0 0 0)
+  )
+  (junction (at 212.09 74.93) (diameter 0) (color 0 0 0 0)
   )
   (junction (at 198.12 154.94) (diameter 0) (color 0 0 0 0)
@@
   (no_connect (at 86.36 182.88))
   (no_connect (at 194.31 36.83))
+  (no_connect (at 196.85 90.17))
   (no_connect (at 106.68 36.83))
   (wire (pts (xy 196.85 97.79) (xy 186.69 97.79))
@@
     (stroke (width 0) (type default) (color 0 0 0 0))
   )
+  (wire (pts (xy 209.55 74.93) (xy 212.09 74.93))
+    (stroke (width 0) (type default) (color 0 0 0 0))
+  )
   (wire (pts (xy 184.15 139.7) (xy 198.12 139.7))
     (stroke (width 0) (type default) (color 0 0 0 0))
@@
     (stroke (width 0) (type default) (color 0 0 0 0))
   )
+  (wire (pts (xy 229.87 87.63) (xy 227.33 87.63))
+    (stroke (width 0) (type default) (color 0 0 0 0))
+  )
   (wire (pts (xy 106.68 39.37) (xy 116.84 39.37))
     (stroke (width 0) (type default) (color 0 0 0 0))
@@
     (stroke (width 0) (type default) (color 0 0 0 0))
   )
+  (wire (pts (xy 227.33 97.79) (xy 229.87 97.79))
+    (stroke (width 0) (type default) (color 0 0 0 0))
+  )
   (wire (pts (xy 102.87 154.94) (xy 118.11 154.94))
     (stroke (width 0) (type default) (color 0 0 0 0))
@@
     (stroke (width 0) (type default) (color 0 0 0 0))
   )
+  (wire (pts (xy 229.87 93.98) (xy 227.33 93.98))
+    (stroke (width 0) (type default) (color 0 0 0 0))
+  )
+  (wire (pts (xy 229.87 97.79) (xy 229.87 100.33))
+    (stroke (width 0) (type default) (color 0 0 0 0))
+  )
   (wire (pts (xy 189.23 142.24) (xy 189.23 127))
     (stroke (width 0) (type default) (color 0 0 0 0))
   )
+  (wire (pts (xy 227.33 85.09) (xy 229.87 85.09))
+    (stroke (width 0) (type default) (color 0 0 0 0))
+  )
   (wire (pts (xy 187.96 153.67) (xy 187.96 166.37))
     (stroke (width 0) (type default) (color 0 0 0 0))
@@
     (stroke (width 0) (type default) (color 0 0 0 0))
   )
+  (wire (pts (xy 229.87 91.44) (xy 229.87 93.98))
+    (stroke (width 0) (type default) (color 0 0 0 0))
+  )
   (wire (pts (xy 72.39 74.93) (xy 71.12 76.2))
     (stroke (width 0) (type default) (color 0 0 0 0))
@@
     (stroke (width 0) (type default) (color 0 0 0 0))
   )
+  (wire (pts (xy 229.87 100.33) (xy 227.33 100.33))
+    (stroke (width 0) (type default) (color 0 0 0 0))
+  )
   (wire (pts (xy 109.22 127) (xy 115.57 127))
     (stroke (width 0) (type default) (color 0 0 0 0))
   )
+  (wire (pts (xy 212.09 105.41) (xy 212.09 106.68))
+    (stroke (width 0) (type default) (color 0 0 0 0))
+  )
   (wire (pts (xy 212.09 80.01) (xy 212.09 74.93))
     (stroke (width 0) (type default) (color 0 0 0 0))
@@
     (stroke (width 0) (type default) (color 0 0 0 0))
   )
+  (wire (pts (xy 229.87 85.09) (xy 229.87 87.63))
+    (stroke (width 0) (type default) (color 0 0 0 0))
+  )
   (wire (pts (xy 102.87 157.48) (xy 107.95 152.4))
     (stroke (width 0) (type default) (color 0 0 0 0))
@@
     (stroke (width 0) (type default) (color 0 0 0 0))
   )
+  (wire (pts (xy 209.55 80.01) (xy 209.55 74.93))
+    (stroke (width 0) (type default) (color 0 0 0 0))
+  )
   (wire (pts (xy 104.14 163.83) (xy 193.04 163.83))
+    (stroke (width 0) (type default) (color 0 0 0 0))
+  )
+  (wire (pts (xy 227.33 91.44) (xy 229.87 91.44))
     (stroke (width 0) (type default) (color 0 0 0 0))
   )
@@
       (effects (font (size 1.27 1.27)) (justify left))
     )
-    (property "Footprint" "Capacitor_SMD:C_0603_1608Metric" (id 2) (at 54.61 41.91 0)
+    (property "Footprint" "Capacitor_SMD:C_0402_1005Metric" (id 2) (at 54.61 41.91 0)
       (effects (font (size 1.27 1.27)) hide)
     )
@@
       (effects (font (size 1.27 1.27)) (justify left))
     )
-    (property "Footprint" "Capacitor_SMD:C_0603_1608Metric" (id 2) (at 40.64 41.91 0)
+    (property "Footprint" "Capacitor_SMD:C_0402_1005Metric" (id 2) (at 40.64 41.91 0)
       (effects (font (size 1.27 1.27)) hide)
     )
@@
       (effects (font (size 1.27 1.27)) (justify left))
     )
-    (property "Footprint" "Capacitor_SMD:C_1206_3216Metric" (id 2) (at 27.94 41.91 0)
+    (property "Footprint" "Capacitor_SMD:C_0805_2012Metric" (id 2) (at 27.94 41.91 0)
       (effects (font (size 1.27 1.27)) hide)
     )
@@
       (effects (font (size 1.27 1.27)) (justify left))
     )
-    (property "Footprint" "Capacitor_SMD:C_0603_1608Metric" (id 2) (at 209.55 134.62 0)
+    (property "Footprint" "Capacitor_SMD:C_0402_1005Metric" (id 2) (at 209.55 134.62 0)
       (effects (font (size 1.27 1.27)) hide)
     )
@@
       (effects (font (size 1.27 1.27)) (justify left))
     )
-    (property "Footprint" "Capacitor_SMD:C_0603_1608Metric" (id 2) (at 242.57 22.86 0))
+    (property "Footprint" "Capacitor_SMD:C_0402_1005Metric" (id 2) (at 242.57 22.86 0))
     (property "Datasheet" "~" (id 3) (at 238.76 33.02 0)
       (effects (font (size 1.27 1.27)) hide)
@@
     (property "Datasheet" "" (id 3) (at 86.36 147.32 0)
       (effects (font (size 1.524 1.524)))
+    )
+    (property "MPN" "EXB-2HV470JV" (id 4) (at 86.36 147.32 0)
+      (effects (font (size 1.27 1.27)) hide)
     )
     (pin "1")
@@
     (pin "1")
   )
+  (symbol (lib_id "power:GND") (at 212.09 106.68 0) (unit 1)
+    (in_bom yes) (on_board yes)
+    (property "Reference" "#PWR0109" (id 0) (at 212.09 113.03 0)
+      (effects (font (size 1.27 1.27)) hide)
+    )
+    (property "Value" "GND" (id 1) (at 212.217 111.0742 0))
+    (property "Footprint" "" (id 2) (at 212.09 106.68 0)
+      (effects (font (size 1.27 1.27)) hide)
+    )
+    (property "Datasheet" "" (id 3) (at 212.09 106.68 0)
+      (effects (font (size 1.27 1.27)) hide)
+    )
+    (pin "1")
+  )
   (symbol (lib_id "Sensor_Pressure:MS5525DSO") (at 212.09 92.71 0) (unit 1)
     (in_bom yes) (on_board yes) (fields_autoplaced)
@@
       (effects (font (size 1.27 1.27)) (justify left))
     )
-    (property "Footprint" "SapphineMinimal:TE_MS5525DSO-DBxxxyS" (id 2) (at 212.09 106.68 0)
+    (property "Footprint" "Sapphire:TE_5525DSO-DB001DS" (id 2) (at 212.09 106.68 0)
       (effects (font (size 1.27 1.27)) hide)
     )
     (property "Datasheet" "https://www.te.com/commerce/DocumentDelivery/DDEController?Action=srchrtrv&DocNm=MS5525DSO&DocType=DS&DocLang=English" (id 3) (at 212.09 109.22 0)
+      (effects (font (size 1.27 1.27)) hide)
+    )
+    (property "Description" "Pressure Sensor 1PSI (6.89kPa) Differential Male - 0.12\" (3mm) Tube, Dual 24 b 14-SMD Module" (id 4) (at 212.09 93.98 0)
+      (effects (font (size 1.27 1.27)) hide)
+    )
+    (property "MPN" "5525DSO-DB001DS" (id 5) (at 212.09 92.71 0)
       (effects (font (size 1.27 1.27)) hide)
     )
@@
       (effects (font (size 1.27 1.27)) (justify left))
     )
-    (property "Footprint" "Capacitor_SMD:C_0603_1608Metric" (id 2) (at 246.38 67.31 0))
+    (property "Footprint" "Capacitor_SMD:C_0402_1005Metric" (id 2) (at 246.38 67.31 0))
     (property "Datasheet" "~" (id 3) (at 242.57 77.47 0)
       (effects (font (size 1.27 1.27)) hide)
@@
       (effects (font (size 1.524 1.524)))
     )
-    (pin "1")
+    (property "Description" "Accelerometer X, Y, Z Axis ±2g, 4g, 8g 25Hz ~ 500Hz 16-LGA (3x3)" (id 4) (at 118.11 139.7 0)
+      (effects (font (size 1.27 1.27)) hide)
+    )
+    (property "MPN" "LIS331DLHTR" (id 5) (at 118.11 139.7 0)
+      (effects (font (size 1.27 1.27)) hide)
+    )
+    (pin "1")
