File: DS3231_sch.kicad_sch (KiCad schematic)
At the start: 6 parts, among them SW802 EVQP7C01P, U802 DS3231SN

Commit message: Partial Routing
Parts:
- added R816, R817: 47, Resistor_SMD:R_0603_1608Metric, symbol Device:R_US
- C811: MPN CL10B104KA8NNNC -> CL05A104KA5NNNC
Connections:
- net I2C_SCL: now also R817.2; no longer U802.16 (SCL)
- net I2C_SDA: now also R816.2; no longer U802.15 (SDA)
- new net: R816.1, U802.15 (SDA)
- new net: R817.1, U802.16 (SCL)
Changed lines of the file:
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@@
+    (stroke (width 0) (type default) (color 0 0 0 0))
+  )
+  (wire (pts (xy 106.68 73.66) (xy 120.65 73.66))
     (stroke (width 0) (type default) (color 0 0 0 0))
   )
@@
     (stroke (width 0) (type default) (color 0 0 0 0))
   )
-  (wire (pts (xy 92.71 73.66) (xy 120.65 73.66))
+  (wire (pts (xy 92.71 73.66) (xy 99.06 73.66))
     (stroke (width 0) (type default) (color 0 0 0 0))
   )
@@
     (stroke (width 0) (type default) (color 0 0 0 0))
   )
+  (wire (pts (xy 106.6357 76.2) (xy 120.65 76.2))
+    (stroke (width 0) (type default) (color 0 0 0 0))
+  )
   (wire (pts (xy 146.05 73.66) (xy 147.32 73.66))
     (stroke (width 0) (type default) (color 0 0 0 0))
@@
     (stroke (width 0) (type default) (color 0 0 0 0))
   )
-  (wire (pts (xy 92.71 76.2) (xy 120.65 76.2))
+  (wire (pts (xy 92.71 76.2) (xy 99.0157 76.2))
     (stroke (width 0) (type default) (color 0 0 0 0))
   )
@@
     (pin "2")
   )
+  (symbol (lib_id "Device:R_US") (at 102.8257 76.2 270) (unit 1)
+    (in_bom yes) (on_board yes)
+    (property "Reference" "R816" (id 0) (at 99.0157 74.93 90))
+    (property "Value" "47" (id 1) (at 105.3657 74.93 90))
+    (property "Footprint" "Resistor_SMD:R_0603_1608Metric" (id 2) (at 102.5717 77.216 90)
+      (effects (font (size 1.27 1.27)) hide)
+    )
+    (property "Datasheet" "~" (id 3) (at 102.8257 76.2 0)
+      (effects (font (size 1.27 1.27)) hide)
+    )
+    (property "Description" "47 Ohms ±1% 0.1W, 1/10W Chip Resistor 0603" (id 4) (at 102.8257 76.2 0)
+      (effects (font (size 1.27 1.27)) hide)
+    )
+    (property "MPN" "CRCW060347R0FKEAC" (id 5) (at 102.8257 76.2 0)
+      (effects (font (size 1.27 1.27)) hide)
+    )
+    (pin "1")
+    (pin "2")
+  )
   (symbol (lib_id "Device:C_Small") (at 161.29 62.23 0) (unit 1)
     (in_bom yes) (on_board yes)
@@
       (effects (font (size 1.27 1.27)) hide)
     )
-    (property "MPN" "CL10B104KA8NNNC" (id 5) (at 161.29 62.23 0)
+    (property "MPN" "CL05A104KA5NNNC" (id 5) (at 161.29 62.23 0)
       (effects (font (size 1.27 1.27)) hide)
     )
@@
     (pin "9")
   )
+  (symbol (lib_id "Device:R_US") (at 102.87 73.66 270) (unit 1)
+    (in_bom yes) (on_board yes)
+    (property "Reference" "R817" (id 0) (at 99.06 72.39 90))
+    (property "Value" "47" (id 1) (at 105.41 72.39 90))
+    (property "Footprint" "Resistor_SMD:R_0603_1608Metric" (id 2) (at 102.616 74.676 90)
+      (effects (font (size 1.27 1.27)) hide)
+    )
+    (property "Datasheet" "~" (id 3) (at 102.87 73.66 0)
+      (effects (font (size 1.27 1.27)) hide)
+    )
+    (property "Description" "47 Ohms ±1% 0.1W, 1/10W Chip Resistor 0603" (id 4) (at 102.87 73.66 0)
+      (effects (font (size 1.27 1.27)) hide)
+    )
+    (property "MPN" "CRCW060347R0FKEAC" (id 5) (at 102.87 73.66 0)
+      (effects (font (size 1.27 1.27)) hide)
+    )
+    (pin "1")
+    (pin "2")
+  )
   (symbol (lib_id "power:GND") (at 133.35 104.14 0) (unit 1)

Commit message: Added slot for wiring
Parts:
- R816, R817: Manufacturer (none) -> Vishay
Changed lines of the file:
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@@
+      (effects (font (size 1.27 1.27)) hide)
+    )
+    (property "Manufacturer" "Vishay" (id 6) (at 102.8257 76.2 0)
       (effects (font (size 1.27 1.27)) hide)
     )
@@
       (effects (font (size 1.27 1.27)) hide)
     )
+    (property "Manufacturer" "Vishay" (id 6) (at 102.87 73.66 0)
+      (effects (font (size 1.27 1.27)) hide)
+    )

Commit message: OSH_ParkM2R3
Parts:
- R816, R817: Populate (none) -> 1
Changed lines of the file:
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@@
+      (effects (font (size 1.27 1.27)) hide)
+    )
+    (property "Populate" "1" (id 7) (at 102.8257 76.2 0)
       (effects (font (size 1.27 1.27)) hide)
     )
@@
       (effects (font (size 1.27 1.27)) hide)
     )
+    (property "Populate" "1" (id 7) (at 102.87 73.66 0)
+      (effects (font (size 1.27 1.27)) hide)
+    )

Commit message: Board ready for final check
Parts:
- C811: footprint Capacitor_SMD:C_0603_1608Metric -> Capacitor_SMD:C_0402_1005Metric
- SW802: footprint SapphineMinimal:EVQP7C01P -> Sapphire:EVQP7C01P_HandSolder; symbol EVQP7C01P:EVQP7C01P -> sapphireMini:EVQP7C01P
Other:
- note added: "DS3231 address 0x68"
Changed lines of the file:
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@@
     (stroke (width 0) (type default) (color 0 0 0 0))
+  )
+  (text "DS3231 address 0x68" (at 94.1693 51.1348 0)
+    (effects (font (size 1.27 1.27)) (justify left bottom))
   )
   (text "DS3231S.  Be sure to avoid DS3231M version of chip \nwhich does not have precision clock output.\nSee datasheet on handling (avoid excessive shocks).\n"
@@
       (effects (font (size 1.27 1.27)) (justify left))
     )
-    (property "Footprint" "Capacitor_SMD:C_0603_1608Metric" (id 2) (at 161.29 62.23 0)
+    (property "Footprint" "Capacitor_SMD:C_0402_1005Metric" (id 2) (at 161.29 62.23 0)
       (effects (font (size 1.27 1.27)) hide)
     )
@@
     (pin "1")
   )
-  (symbol (lib_id "EVQP7C01P:EVQP7C01P") (at 77.47 100.33 0) (unit 1)
+  (symbol (lib_id "sapphireMini:EVQP7C01P") (at 77.47 100.33 0) (unit 1)
     (in_bom yes) (on_board yes)
     (property "Reference" "SW802" (id 0) (at 104.14 88.8238 0)
@@
       (effects (font (size 1.524 1.524)))
     )
-    (property "Footprint" "SapphineMinimal:EVQP7C01P" (id 2) (at 91.44 99.06 0)
+    (property "Footprint" "Sapphire:EVQP7C01P_HandSolder" (id 2) (at 91.44 99.06 0)
       (effects (font (size 1.524 1.524)) hide)
     )
