File: SapphineMinimal.kicad_sch (KiCad schematic)
At the start: 6 parts

Commit message: End of Weekend
Other:
- removed sheet RV8803
- added sheet DS3231 (DS3231_sch.kicad_sch)
- sheet Sapphire_Proc ports: added RESET, SPARE; removed CLK_EVI

Commit message: Midst of pretying layout
Other:
- sheet Sapphire_WiFi ports: added SPARE; removed none
Changed lines of the file:
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@@
+    (stroke (width 0) (type default) (color 0 0 0 0))
+  )
+  (wire (pts (xy 226.06 105.41) (xy 226.06 130.81))
     (stroke (width 0) (type default) (color 0 0 0 0))
   )
@@
     (stroke (width 0) (type default) (color 0 0 0 0))
   )
+  (wire (pts (xy 224.79 104.14) (xy 226.06 105.41))
+    (stroke (width 0) (type default) (color 0 0 0 0))
+  )
   (wire (pts (xy 171.45 83.82) (xy 181.61 83.82))
     (stroke (width 0) (type default) (color 0 0 0 0))
@@
     (stroke (width 0) (type default) (color 0 0 0 0))
   )
-  (wire (pts (xy 107.95 43.18) (xy 120.65 43.18))
-    (stroke (width 0) (type default) (color 0 0 0 0))
-  )
   (wire (pts (xy 76.2 116.84) (xy 107.95 116.84))
     (stroke (width 0) (type default) (color 0 0 0 0))
@@
   )
   (wire (pts (xy 219.71 57.15) (xy 238.76 57.15))
+    (stroke (width 0) (type default) (color 0 0 0 0))
+  )
+  (wire (pts (xy 171.45 104.14) (xy 224.79 104.14))
     (stroke (width 0) (type default) (color 0 0 0 0))
   )
@@
       (effects (font (size 1.27 1.27)) (justify left))
     )
-    (pin "SPARE" output (at 120.65 43.18 180)
-      (effects (font (size 1.27 1.27)) (justify left))
+    (pin "SPARE" output (at 171.45 104.14 0)
+      (effects (font (size 1.27 1.27)) (justify right))
     )
   )
@@
     (pin "SPI2_MOSI" input (at 181.61 153.67 180)
       (effects (font (size 1.27 1.27)) (justify left))
+    )
+    (pin "SPARE" input (at 226.06 130.81 90)
+      (effects (font (size 1.27 1.27)) (justify right))
     )
   )
@@
       (reference "R604") (unit 1) (value "47") (footprint "Resistor_SMD:R_0603_1608Metric")
     )
+    (path "/00000000-0000-0000-0000-000063a74ef2/41dc9c4c-f9fb-4724-aea9-3a0ceea817ae"
+      (reference "R605") (unit 1) (value "47") (footprint "Resistor_SMD:R_0603_1608Metric")
+    )
     (path "/00000000-0000-0000-0000-000063a74ef2/6d43920e-21c5-441e-8415-c5dfb7b75379"

Commit message: OSH_ParkM2R3
Parts:
- FID101, FID102, FID103, FID104, FID105, FID106: Populate (none) -> 0
Changed lines of the file:
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@@
+      (effects (font (size 1.27 1.27)) hide)
+    )
+    (property "Populate" "0" (id 4) (at 255.27 48.26 0)
       (effects (font (size 1.27 1.27)) hide)
     )
@@
       (effects (font (size 1.27 1.27)) hide)
     )
+    (property "Populate" "0" (id 4) (at 255.27 25.4 0)
+      (effects (font (size 1.27 1.27)) hide)
+    )
   )
   (symbol (lib_id "Mechanical:Fiducial") (at 255.27 34.29 0) (unit 1)
@@
       (effects (font (size 1.27 1.27)) hide)
     )
+    (property "Populate" "0" (id 4) (at 255.27 34.29 0)
+      (effects (font (size 1.27 1.27)) hide)
+    )
   )
   (symbol (lib_id "Mechanical:Fiducial") (at 255.27 43.18 0) (unit 1)
@@
       (effects (font (size 1.27 1.27)) hide)
     )
+    (property "Populate" "0" (id 4) (at 255.27 43.18 0)
+      (effects (font (size 1.27 1.27)) hide)
+    )
   )
   (symbol (lib_id "Mechanical:Fiducial") (at 255.27 29.845 0) (unit 1)
@@
       (effects (font (size 1.27 1.27)) hide)
     )
+    (property "Populate" "0" (id 4) (at 255.27 29.845 0)
+      (effects (font (size 1.27 1.27)) hide)
+    )
   )
   (symbol (lib_id "Mechanical:Fiducial") (at 255.27 38.735 0) (unit 1)
@@
     )
     (property "Datasheet" "~" (id 3) (at 255.27 38.735 0)
+      (effects (font (size 1.27 1.27)) hide)
+    )
+    (property "Populate" "0" (id 4) (at 255.27 38.735 0)
       (effects (font (size 1.27 1.27)) hide)
     )
@@
     )
     (path "/00000000-0000-0000-0000-00005e3fe689/00000000-0000-0000-0000-00005e66dbe9"
-      (reference "IC201") (unit 1) (value "DLHR-F50D-E1BD-C-NAV8") (footprint "Sapphire:DLHRF50DE1BDCNAV8")
+      (reference "IC201") (unit 1) (value "DNP DLHR-F50D-E1BD-C-NAV8") (footprint "Sapphire:DLHRF50DE1BDCNAV8")
     )
     (path "/00000000-0000-0000-0000-00005e3fe3dd/28ca0051-4e73-486f-a8fb-1e04cfc47f1d"
@@
     )
     (path "/00000000-0000-0000-0000-00005e3fe93a/00000000-0000-0000-0000-000063937b6f"
-      (reference "J401") (unit 1) (value "Conn_01x01_Male") (footprint "TestPoint:TestPoint_Pad_1.0x1.0mm")
+      (reference "J401") (unit 1) (value "DNP Conn_01x01_Male") (footprint "TestPoint:TestPoint_Pad_1.0x1.0mm")
     )
     (path "/00000000-0000-0000-0000-00005e3fe93a/6bda1ba2-5697-4584-8671-03daa411d89e"
@@
     )
     (path "/00000000-0000-0000-0000-000063357571/00000000-0000-0000-0000-0000635a1b6c"
-      (reference "J802") (unit 1) (value "Conn_02x05_Odd_Even") (footprint "Sapphire:3220-10-0100-00")
+      (reference "J802") (unit 1) (value "DNP Conn_02x05_Odd_Even") (footprint "Sapphire:3220-10-0100-00")
     )
     (path "/00000000-0000-0000-0000-000063357571/00000000-0000-0000-0000-000063815981"
-      (reference "J803") (unit 1) (value "Conn_02x05_Odd_Even") (footprint "Sapphire:3220-10-0100-00")
+      (reference "J803") (unit 1) (value "DNP Conn_02x05_Odd_Even") (footprint "Sapphire:3220-10-0100-00")
     )
     (path "/00000000-0000-0000-0000-000063357571/00000000-0000-0000-0000-0000637481f1"
@@
     )
     (path "/00000000-0000-0000-0000-000063a74ef2/00000000-0000-0000-0000-000063a75a3b"
-      (reference "M701") (unit 1) (value "AdafruitWINC1500") (footprint "Connector_PinHeader_2.54mm:PinHeader_1x13_P2.54mm_Vertical")
+      (reference "M701") (unit 1) (value "DNP AdafruitWINC1500") (footprint "Connector_PinHeader_2.54mm:PinHeader_1x13_P2.54mm_Vertical")
     )
     (path "/00000000-0000-0000-0000-00005e3fe3dd/00000000-0000-0000-0000-00005e41cace"
-      (reference "Q501") (unit 1) (value "BC857BS") (footprint "Package_TO_SOT_SMD:SOT-363_SC-70-6")
+      (reference "Q501") (unit 1) (value "BC857BDW1T1G") (footprint "Package_TO_SOT_SMD:SOT-363_SC-70-6")
     )
     (path "/00000000-0000-0000-0000-00005e3fe3dd/00000000-0000-0000-0000-00005e41cac8"
-      (reference "Q501") (unit 2) (value "BC857BS") (footprint "Package_TO_SOT_SMD:SOT-363_SC-70-6")
+      (reference "Q501") (unit 2) (value "BC857BDW1T1G") (footprint "Package_TO_SOT_SMD:SOT-363_SC-70-6")
     )
     (path "/00000000-0000-0000-0000-00005e3fe3dd/72bdceb4-14fa-4bbc-ad1d-2262438e77f3"
@@
     )
     (path "/00000000-0000-0000-0000-000063a74ef2/770a810f-7184-4b44-9425-19097f9992b5"
-      (reference "R602") (unit 1) (value "0") (footprint "Resistor_SMD:R_0603_1608Metric")
+      (reference "R602") (unit 1) (value "DNP 0") (footprint "Resistor_SMD:R_0603_1608Metric")
     )
     (path "/00000000-0000-0000-0000-000063a74ef2/c26ca922-835a-4202-97d2-3b260d7d3c1c"
@@
     )
     (path "/00000000-0000-0000-0000-000063a74ef2/6d43920e-21c5-441e-8415-c5dfb7b75379"
-      (reference "R702") (unit 1) (value "47") (footprint "Resistor_SMD:R_0603_1608Metric")
+      (reference "R702") (unit 1) (value "DNP 47") (footprint "Resistor_SMD:R_0603_1608Metric")
     )
     (path "/00000000-0000-0000-0000-000063a74ef2/44066c90-8c1b-4164-acc8-5fad27e22e40"
-      (reference "R703") (unit 1) (value "47") (footprint "Resistor_SMD:R_0603_1608Metric")
+      (reference "R703") (unit 1) (value "DNP 47") (footprint "Resistor_SMD:R_0603_1608Metric")
     )
     (path "/00000000-0000-0000-0000-000063357571/00000000-0000-0000-0000-0000634d9925"
@@
     )
     (path "/00000000-0000-0000-0000-00005e3fe689/3a65f7fd-136d-4cc0-bad7-5b08a056ab22"
-      (reference "U201") (unit 1) (value "LIS2DH12TR") (footprint "Sapphire:LIS2DH12TR")
+      (reference "U201") (unit 1) (value "LIS2HH12TR") (footprint "Sapphire:LIS2DH12TR")
     )
     (path "/00000000-0000-0000-0000-00005e3fe689/00000000-0000-0000-0000-0000639b31d6"

Commit message: Board ready for final check
Parts:
- added Ha101, Hb101, Hc101: MountingHole, MountingHole:MountingHole_3.2mm_M3, symbol Mechanical:MountingHole
- FID101, FID102, FID103, FID104, FID105, FID106: now left out of the parts list
Connections:
- no-connect marks 1 -> 2
Other:
- sheet SapphireMini_DLHR ports: added 32KHz, SPARE; removed none
- sheet SapphireMini_GNSS ports: added none; removed P3V3
- sheet SapphireMini_Power ports: added VBAT_EN; removed none
