File: SapphireMini_GNSS.kicad_sch (KiCad schematic)
At the start: 13 parts, among them J401 Conn_01x01_Male, J402 Conn_01x04_Male, J403 ExtPPS, U402 SAM-M8Q-0-10

Commit message: InProgress
Parts:
- gave numbers to parts that had none: 5
Changed lines of the file:
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@@
   (symbol (lib_id "Device:R_Small_US") (at 111.76 118.11 180) (unit 1)
     (in_bom yes) (on_board yes)
-    (property "Reference" "R?" (id 0) (at 110.49 115.57 0)
+    (property "Reference" "R403" (id 0) (at 110.49 115.57 0)
       (effects (font (size 1.27 1.27)) (justify left))
     )
@@
   (symbol (lib_id "Device:LED") (at 104.14 107.95 90) (unit 1)
     (in_bom yes) (on_board yes)
-    (property "Reference" "D?" (id 0) (at 105.41 104.14 90)
+    (property "Reference" "D401" (id 0) (at 105.41 104.14 90)
       (effects (font (size 1.27 1.27)) (justify right))
     )
@@
   (symbol (lib_id "power:GND") (at 111.76 124.46 0) (unit 1)
     (in_bom yes) (on_board yes)
-    (property "Reference" "#PWR?" (id 0) (at 111.76 130.81 0)
+    (property "Reference" "#PWR0112" (id 0) (at 111.76 130.81 0)
       (effects (font (size 1.27 1.27)) hide)
     )
@@
   (symbol (lib_id "Device:R_Small_US") (at 104.14 118.11 180) (unit 1)
     (in_bom yes) (on_board yes)
-    (property "Reference" "R?" (id 0) (at 101.6 116.84 0)
+    (property "Reference" "R402" (id 0) (at 101.6 116.84 0)
       (effects (font (size 1.27 1.27)) (justify left))
     )
@@
   (symbol (lib_id "power:GND") (at 104.14 124.46 0) (unit 1)
     (in_bom yes) (on_board yes)
-    (property "Reference" "#PWR?" (id 0) (at 104.14 130.81 0)
+    (property "Reference" "#PWR0111" (id 0) (at 104.14 130.81 0)
       (effects (font (size 1.27 1.27)) hide)
     )
@@
   (symbol (lib_id "Device:LED") (at 111.76 107.95 90) (unit 1)
     (in_bom yes) (on_board yes)
-    (property "Reference" "D?" (id 0) (at 113.03 104.14 90)
+    (property "Reference" "D402" (id 0) (at 113.03 104.14 90)
       (effects (font (size 1.27 1.27)) (justify right))
     )
@@
   (symbol (lib_id "Device:R_Small_US") (at 115.57 118.11 180) (unit 1)
     (in_bom yes) (on_board yes)
-    (property "Reference" "R?" (id 0) (at 118.11 115.57 0)
-      (effects (font (size 1.27 1.27)) (justify left))
-    )
+    (property "Reference" "R404" (id 0) (at 118.11 115.57 0)
+      (effects (font (size 1.27 1.27)) (justify left))
+    )

Commit message: OSH_ParkM2R3
Parts:
- FB401, FB403, R401, U402: Populate (none) -> 1
- J401: value Conn_01x01_Male -> DNP Conn_01x01_Male; Populate (none) -> 0
- J403: Populate (none) -> 0
Changed lines of the file:
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@@
+      (effects (font (size 1.27 1.27)) hide)
+    )
+    (property "Populate" "1" (id 11) (at 156.21 102.87 0)
       (effects (font (size 1.27 1.27)) hide)
     )
@@
       (effects (font (size 1.27 1.27)) (justify right))
     )
-    (property "Value" "Conn_01x01_Male" (id 1) (at 207.7212 113.6142 0)
+    (property "Value" "DNP Conn_01x01_Male" (id 1) (at 207.7212 113.6142 0)
       (effects (font (size 1.27 1.27)) (justify right) hide)
     )
@@
       (effects (font (size 1.27 1.27)) hide)
     )
+    (property "Populate" "0" (id 6) (at 207.01 113.03 0)
+      (effects (font (size 1.27 1.27)) hide)
+    )
     (pin "1")
   )
@@
       (effects (font (size 1.27 1.27)) hide)
     )
+    (property "Populate" "1" (id 6) (at 45.72 85.09 0)
+      (effects (font (size 1.27 1.27)) hide)
+    )
     (pin "1")
     (pin "2")
@@
     )
     (property "MPN" "EXB-2HV470JV" (id 4) (at 52.07 80.01 0)
+      (effects (font (size 1.27 1.27)) hide)
+    )
+    (property "Populate" "1" (id 5) (at 52.07 80.01 0)
       (effects (font (size 1.27 1.27)) hide)
     )
@@
       (effects (font (size 1.27 1.27)) hide)
     )
+    (property "Populate" "1" (id 6) (at 68.58 46.99 0)
+      (effects (font (size 1.27 1.27)) hide)
+    )
     (pin "1")
     (pin "2")
@@
       (effects (font (size 1.27 1.27)) hide)
     )
+    (property "Populate" "0" (id 4) (at 134.62 63.5 0)
+      (effects (font (size 1.27 1.27)) hide)
+    )

Commit message: Board ready for final check
Parts:
- D402: symbol Device:LED -> sapphireMini:LED_G
Connections:
- net TIMEPULSE: now also D402.1 (A); no longer D402.2 (A)
- net at R403.2, R404.2: now also D402.2 (K); no longer D402.1 (K)
- no-connect marks 3 -> 8
Changed lines of the file:
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@@
     (comment 2 "Markup copy w/ errors!")
   )
+  (junction (at 88.392 46.99) (diameter 0) (color 0 0 0 0)
+  )
   (junction (at 95.25 90.17) (diameter 0) (color 0 0 0 0)
   )
@@
   (junction (at 111.76 120.65) (diameter 0) (color 0 0 0 0)
   )
-  (no_connect (at 78.74 80.01))
+  (no_connect (at 40.64 105.41))
+  (no_connect (at 40.64 100.33))
+  (no_connect (at 78.74 95.25))
+  (no_connect (at 78.74 105.41))
+  (no_connect (at 78.74 100.33))
+  (no_connect (at 40.64 95.25))
   (no_connect (at 177.8 107.95))
   (no_connect (at 177.8 105.41))
@@
     (stroke (width 0) (type default) (color 0 0 0 0))
   )
-  (wire (pts (xy 72.39 46.99) (xy 95.25 46.99))
+  (wire (pts (xy 72.39 46.99) (xy 88.392 46.99))
     (stroke (width 0) (type default) (color 0 0 0 0))
   )
@@
   )
   (wire (pts (xy 111.76 100.33) (xy 135.89 100.33))
+    (stroke (width 0) (type default) (color 0 0 0 0))
+  )
+  (wire (pts (xy 88.392 46.99) (xy 95.25 46.99))
     (stroke (width 0) (type default) (color 0 0 0 0))
   )
@@
   (symbol (lib_id "Device:LED") (at 104.14 107.95 90) (unit 1)
     (in_bom yes) (on_board yes)
-    (property "Reference" "D401" (id 0) (at 105.41 104.14 90)
+    (property "Reference" "D401" (id 0) (at 105.2345 101.3842 0)
       (effects (font (size 1.27 1.27)) (justify right))
     )
@@
     (pin "3")
     (pin "4")
+  )
+  (symbol (lib_id "power:PWR_FLAG") (at 88.392 46.99 0) (unit 1)
+    (in_bom yes) (on_board yes) (fields_autoplaced)
+    (property "Reference" "#FLG0102" (id 0) (at 88.392 45.085 0)
+      (effects (font (size 1.27 1.27)) hide)
+    )
+    (property "Value" "PWR_FLAG" (id 1) (at 88.392 43.4142 0))
+    (property "Footprint" "" (id 2) (at 88.392 46.99 0)
+      (effects (font (size 1.27 1.27)) hide)
+    )
+    (property "Datasheet" "~" (id 3) (at 88.392 46.99 0)
+      (effects (font (size 1.27 1.27)) hide)
+    )
+    (pin "1")
   )
   (symbol (lib_id "power:GND") (at 111.76 124.46 0) (unit 1)
@@
     (pin "9")
   )
-  (symbol (lib_id "Device:LED") (at 111.76 107.95 90) (unit 1)
-    (in_bom yes) (on_board yes)
-    (property "Reference" "D402" (id 0) (at 113.03 104.14 90)
+  (symbol (lib_id "sapphireMini:LED_G") (at 111.76 107.95 90) (unit 1)
+    (in_bom yes) (on_board yes)
+    (property "Reference" "D402" (id 0) (at 113.1004 101.2372 0)
       (effects (font (size 1.27 1.27)) (justify right))
     )
@@
       (effects (font (size 1.27 1.27)) hide)
     )
-    (property "Datasheet" "https://media.digikey.com/pdf/Data%20Sheets/Lite-On%20PDFs/LTST-S220GKT.pdf" (id 3) (at 111.76 107.95 0)
-      (effects (font (size 1.27 1.27)) hide)
-    )
+    (property "Datasheet" "~" (id 3) (at 111.76 107.95 0)
+      (effects (font (size 1.27 1.27)) hide)
+    )
