File: SapphireMini_Proc.kicad_sch (KiCad schematic)
At the start: 38 parts, among them J801 USB_B_Micro, J802 Conn_02x05_Odd_Even, J803 Conn_02x05_Odd_Even, J805 Conn_01x04_Male, SW701 EVQP7C01P, SW801 EVQP7C01P, U801 ATSAMD21G18A-A

Commit message: End of Weekend
Parts:
- removed SW701: EVQP7C01P, Sapphire:EVQP7C01P, symbol sapphireMini:EVQP7C01P
Connections:
- net CLK_EVI renamed SPARE
Other:
- note added: "Consider resistor on 32KHz clock line to clean up pulse"
Changed lines of the file:
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@@
   (junction (at 217.17 81.28) (diameter 0) (color 0 0 0 0)
   )
-  (junction (at 26.67 209.55) (diameter 0) (color 0 0 0 0)
-  )
   (junction (at 49.53 208.28) (diameter 0) (color 0 0 0 0)
   )
@@
   (junction (at 200.66 105.41) (diameter 0) (color 0 0 0 0)
   )
-  (junction (at 26.67 190.5) (diameter 0) (color 0 0 0 0)
-  )
   (junction (at 245.11 182.88) (diameter 0) (color 0 0 0 0)
   )
   (junction (at 90.17 87.63) (diameter 0) (color 0 0 0 0)
-  )
-  (junction (at 26.67 196.85) (diameter 0) (color 0 0 0 0)
   )
   (no_connect (at 241.3 187.96))
@@
     (stroke (width 0) (type default) (color 0 0 0 0))
   )
-  (wire (pts (xy 26.67 200.66) (xy 26.67 196.85))
-    (stroke (width 0) (type default) (color 0 0 0 0))
-  )
   (wire (pts (xy 212.09 193.04) (xy 204.47 193.04))
     (stroke (width 0) (type default) (color 0 0 0 0))
@@
     (stroke (width 0) (type default) (color 0 0 0 0))
   )
-  (wire (pts (xy 36.83 209.55) (xy 26.67 209.55))
-    (stroke (width 0) (type default) (color 0 0 0 0))
-  )
   (wire (pts (xy 59.69 193.04) (xy 59.69 190.5))
     (stroke (width 0) (type default) (color 0 0 0 0))
@@
     (stroke (width 0) (type default) (color 0 0 0 0))
   )
-  (wire (pts (xy 26.67 196.85) (xy 36.83 196.85))
-    (stroke (width 0) (type default) (color 0 0 0 0))
-  )
   (wire (pts (xy 368.3 162.56) (xy 375.92 162.56))
     (stroke (width 0) (type default) (color 0 0 0 0))
@@
     (stroke (width 0) (type default) (color 0 0 0 0))
   )
-  (wire (pts (xy 36.83 205.74) (xy 36.83 209.55))
-    (stroke (width 0) (type default) (color 0 0 0 0))
-  )
   (wire (pts (xy 303.53 118.11) (xy 299.72 118.11))
     (stroke (width 0) (type default) (color 0 0 0 0))
@@
     (stroke (width 0) (type default) (color 0 0 0 0))
   )
-  (wire (pts (xy 36.83 196.85) (xy 36.83 200.66))
-    (stroke (width 0) (type default) (color 0 0 0 0))
-  )
   (wire (pts (xy 283.21 102.87) (xy 270.51 102.87))
     (stroke (width 0) (type default) (color 0 0 0 0))
@@
     (stroke (width 0) (type default) (color 0 0 0 0))
   )
-  (wire (pts (xy 26.67 190.5) (xy 24.13 190.5))
+  (wire (pts (xy 24.13 190.5) (xy 36.83 190.5))
     (stroke (width 0) (type default) (color 0 0 0 0))
   )
@@
     (stroke (width 0) (type default) (color 0 0 0 0))
   )
-  (wire (pts (xy 26.67 209.55) (xy 26.67 215.9))
-    (stroke (width 0) (type default) (color 0 0 0 0))
-  )
   (wire (pts (xy 369.57 57.15) (xy 375.92 57.15))
     (stroke (width 0) (type default) (color 0 0 0 0))
@@
     (stroke (width 0) (type default) (color 0 0 0 0))
   )
-  (wire (pts (xy 26.67 196.85) (xy 26.67 190.5))
-    (stroke (width 0) (type default) (color 0 0 0 0))
-  )
   (wire (pts (xy 59.69 96.52) (xy 59.69 95.25))
     (stroke (width 0) (type default) (color 0 0 0 0))
@@
     (stroke (width 0) (type default) (color 0 0 0 0))
   )
-  (wire (pts (xy 36.83 190.5) (xy 26.67 190.5))
-    (stroke (width 0) (type default) (color 0 0 0 0))
-  )
   (wire (pts (xy 204.47 203.2) (xy 240.03 203.2))
     (stroke (width 0) (type default) (color 0 0 0 0))
@@
   )
   (wire (pts (xy 74.93 57.15) (xy 73.66 58.42))
-    (stroke (width 0) (type default) (color 0 0 0 0))
-  )
-  (wire (pts (xy 26.67 205.74) (xy 26.67 209.55))
     (stroke (width 0) (type default) (color 0 0 0 0))
   )
@@
     (effects (font (size 2.54 2.54)) (justify left bottom))
   )
+  (text "Consider resistor on 32KHz\nclock line to clean up pulse"
+    (at 29.21 31.75 0)
+    (effects (font (size 1.27 1.27)) (justify left bottom))
+  )
   (text "Place decoupling \nclose to relevant pins" (at 104.14 85.09 0)
     (effects (font (size 1.27 1.27)) (justify left bottom))
@@
     (effects (font (size 1.27 1.27)) (justify right))
   )
+  (hierarchical_label "RESET" (shape input) (at 24.13 190.5 180)
+    (effects (font (size 1.27 1.27)) (justify right))
+  )
   (hierarchical_label "GNSS_EXTINT" (shape output) (at 118.11 111.76 0)
     (effects (font (size 1.27 1.27)) (justify left))
@@
     (effects (font (size 1.27 1.27)) (justify right))
   )
-  (hierarchical_label "CLK_EVI" (shape output) (at 344.17 137.16 180)
+  (hierarchical_label "SPARE" (shape output) (at 344.17 137.16 180)
     (effects (font (size 1.27 1.27)) (justify right))
   )
@@
     (pin "4")
   )
-  (symbol (lib_name "EVQP7C01P_1") (lib_id "sapphireMini:EVQP7C01P") (at 33.02 229.87 90) (unit 1)
-    (in_bom yes) (on_board yes)
-    (property "Reference" "SW701" (id 0) (at 21.5138 203.2 0)
-      (effects (font (size 1.524 1.524)))
-    )
-    (property "Value" "EVQP7C01P" (id 1) (at 24.2062 203.2 0)
-      (effects (font (size 1.524 1.524)))
-    )
-    (property "Footprint" "Sapphire:EVQP7C01P" (id 2) (at 27.305 186.055 90)
-      (effects (font (size 1.524 1.524)) hide)
-    )
-    (property "Datasheet" "" (id 3) (at 33.02 229.87 0)
-      (effects (font (size 1.524 1.524)))
-    )
-    (property "Populate" "1" (id 4) (at 33.02 229.87 0)
-      (effects (font (size 1.27 1.27)) hide)
-    )
-    (property "Description" "Tactile Switch SPST-NO Side Actuated Surface Mount, Right Angle" (id 5) (at 33.02 229.87 0)
-      (effects (font (size 1.27 1.27)) hide)
-    )
-    (property "Digi-Key_PN" "P16765CT-ND" (id 6) (at 33.02 229.87 0)
-      (effects (font (size 1.27 1.27)) hide)
-    )
-    (property "MPN" "EVQ-P7C01P" (id 7) (at 33.02 229.87 0)
-      (effects (font (size 1.27 1.27)) hide)
-    )
-    (property "Distributor" "Digikey" (id 8) (at 33.02 229.87 0)
-      (effects (font (size 1.27 1.27)) hide)
-    )
-    (pin "1")
-    (pin "2")
-    (pin "3")
-    (pin "4")
-  )
   (symbol (lib_id "sapphireMini:EXB-2HV470JV_1") (at 355.6 127 0) (unit 1)
     (in_bom yes) (on_board yes)
@@
     (pin "9")
   )
-  (symbol (lib_id "power:GND") (at 26.67 215.9 0) (unit 1)
-    (in_bom yes) (on_board yes)
-    (property "Reference" "#PWR0105" (id 0) (at 26.67 222.25 0)
-      (effects (font (size 1.27 1.27)) hide)
-    )
-    (property "Value" "GND" (id 1) (at 24.13 219.71 0))
-    (property "Footprint" "" (id 2) (at 26.67 215.9 0)
-      (effects (font (size 1.27 1.27)) hide)
-    )
-    (property "Datasheet" "" (id 3) (at 26.67 215.9 0)
-      (effects (font (size 1.27 1.27)) hide)
-    )
-    (pin "1")
-  )
   (symbol (lib_id "Device:FerriteBead") (at 97.79 52.07 0) (unit 1)

Commit message: OSH_ParkM2R3
Parts:
- C803, FB702, FB801, J801, R809, R810, R811, R812, R813, R841: Populate (none) -> 1
- CR801: Consign (none) -> 500
- J802, J803: value Conn_02x05_Odd_Even -> DNP Conn_02x05_Odd_Even; Populate 1 -> 0
- U801: Consign (none) -> 410; Populate (none) -> 1
Changed lines of the file:
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@@
+      (effects (font (size 1.27 1.27)) hide)
+    )
+    (property "Populate" "1" (id 7) (at 49.53 196.85 0)
       (effects (font (size 1.27 1.27)) hide)
     )
@@
     )
     (property "Manufacturer" "KYOCERA AVX" (id 6) (at 59.69 196.85 0)
+      (effects (font (size 1.27 1.27)) hide)
+    )
+    (property "Populate" "1" (id 7) (at 59.69 196.85 0)
       (effects (font (size 1.27 1.27)) hide)
     )
@@
       (effects (font (size 1.27 1.27)) hide)
     )
+    (property "Populate" "1" (id 6) (at 40.64 190.5 0)
+      (effects (font (size 1.27 1.27)) hide)
+    )
     (pin "1")
     (pin "2")
@@
     )
     (property "Description" "2 kOhms ±1% 0.1W, 1/10W Chip Resistor 0603" (id 6) (at 217.17 87.63 0)
+      (effects (font (size 1.27 1.27)) hide)
+    )
+    (property "Populate" "1" (id 7) (at 217.17 87.63 0)
       (effects (font (size 1.27 1.27)) hide)
     )
@@
     )
     (property "Status" "" (id 13) (at 229.87 187.96 0)
+      (effects (font (size 1.27 1.27)) hide)
+    )
+    (property "Consign" "500" (id 14) (at 229.87 187.96 0)
       (effects (font (size 1.27 1.27)) hide)
     )
@@
     (in_bom yes) (on_board yes)
     (property "Reference" "J802" (id 0) (at 207.01 89.7382 0))
-    (property "Value" "Conn_02x05_Odd_Even" (id 1) (at 212.09 110.49 0))
+    (property "Value" "DNP Conn_02x05_Odd_Even" (id 1) (at 212.09 110.49 0))
     (property "Footprint" "Sapphire:3220-10-0100-00" (id 2) (at 205.74 100.33 0)
       (effects (font (size 1.27 1.27)) hide)
@@
       (effects (font (size 1.27 1.27)) hide)
     )
-    (property "Populate" "1" (id 6) (at 205.74 100.33 0)
+    (property "Populate" "0" (id 6) (at 205.74 100.33 0)
       (effects (font (size 1.27 1.27)) hide)
     )
@@
     (in_bom yes) (on_board yes)
     (property "Reference" "J803" (id 0) (at 207.01 120.2182 0))
-    (property "Value" "Conn_02x05_Odd_Even" (id 1) (at 212.09 140.97 0))
+    (property "Value" "DNP Conn_02x05_Odd_Even" (id 1) (at 212.09 140.97 0))
     (property "Footprint" "Sapphire:3220-10-0100-00" (id 2) (at 205.74 130.81 0)
       (effects (font (size 1.27 1.27)) hide)
@@
       (effects (font (size 1.27 1.27)) hide)
     )
-    (property "Populate" "1" (id 6) (at 205.74 130.81 0)
+    (property "Populate" "0" (id 6) (at 205.74 130.81 0)
       (effects (font (size 1.27 1.27)) hide)
     )
@@
     )
     (property "Manufacturer" "Microchip Technology" (id 6) (at 90.17 147.32 0)
+      (effects (font (size 1.27 1.27)) hide)
+    )
+    (property "Populate" "1" (id 7) (at 90.17 147.32 0)
+      (effects (font (size 1.27 1.27)) hide)
+    )
+    (property "Consign" "410" (id 8) (at 90.17 147.32 0)
       (effects (font (size 1.27 1.27)) hide)
     )
@@
       (effects (font (size 1.27 1.27)) hide)
     )
+    (property "Populate" "1" (id 5) (at 355.6 127 0)
+      (effects (font (size 1.27 1.27)) hide)
+    )
     (pin "1")
     (pin "10")
@@
       (effects (font (size 1.27 1.27)) hide)
     )
+    (property "Populate" "1" (id 7) (at 196.85 198.12 0)
+      (effects (font (size 1.27 1.27)) hide)
+    )
     (pin "1")
     (pin "2")
@@
       (effects (font (size 1.27 1.27)) hide)
     )
+    (property "Populate" "1" (id 6) (at 337.82 67.31 0)
+      (effects (font (size 1.27 1.27)) hide)
+    )
     (pin "1")
     (pin "2")
@@
     )
     (property "MPN" "EXB-2HV470JV" (id 4) (at 355.6 80.01 0)
+      (effects (font (size 1.27 1.27)) hide)
+    )
+    (property "Populate" "1" (id 5) (at 355.6 80.01 0)
       (effects (font (size 1.27 1.27)) hide)
     )
@@
       (effects (font (size 1.27 1.27)) hide)
     )
+    (property "Populate" "1" (id 6) (at 97.79 52.07 0)
+      (effects (font (size 1.27 1.27)) hide)
+    )
     (pin "1")
     (pin "2")
@@
       (effects (font (size 1.27 1.27)) hide)
     )
+    (property "Populate" "1" (id 5) (at 356.87 31.75 0)
+      (effects (font (size 1.27 1.27)) hide)
+    )

Commit message: Board ready for final check
Parts:
- D803: symbol Device:LED -> sapphireMini:LED_G
- SW801: footprint Sapphire:EVQP7C01P -> Sapphire:EVQP7C01P_HandSolder
Connections:
- net GREEN_LED: now also D803.1 (A); no longer D803.2 (A)
- net at R805.1, R806.1: now also D803.2 (K); no longer D803.1 (K)
Changed lines of the file:
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@@
   (junction (at 87.63 87.63) (diameter 0) (color 0 0 0 0)
+  )
+  (junction (at 97.79 61.468) (diameter 0) (color 0 0 0 0)
   )
   (junction (at 299.72 118.11) (diameter 0) (color 0 0 0 0)
@@
     (stroke (width 0) (type default) (color 0 0 0 0))
   )
+  (wire (pts (xy 97.79 61.468) (xy 97.79 71.12))
+    (stroke (width 0) (type default) (color 0 0 0 0))
+  )
   (wire (pts (xy 344.17 115.57) (xy 355.6 115.57))
     (stroke (width 0) (type default) (color 0 0 0 0))
@@
     (stroke (width 0) (type default) (color 0 0 0 0))
   )
-  (wire (pts (xy 97.79 58.42) (xy 97.79 71.12))
+  (wire (pts (xy 97.79 58.42) (xy 97.79 61.468))
     (stroke (width 0) (type default) (color 0 0 0 0))
   )
@@
     (pin "1")
   )
-  (symbol (lib_id "Device:LED") (at 287.02 102.87 180) (unit 1)
+  (symbol (lib_name "LED_1") (lib_id "Device:LED") (at 287.02 102.87 180) (unit 1)
     (in_bom yes) (on_board yes)
     (property "Reference" "D802" (id 0) (at 286.0294 99.8728 0)
@@
     (pin "2")
   )
-  (symbol (lib_id "Device:LED") (at 287.02 118.11 180) (unit 1)
+  (symbol (lib_id "sapphireMini:LED_G") (at 287.02 118.11 180) (unit 1)
     (in_bom yes) (on_board yes)
     (property "Reference" "D803" (id 0) (at 286.0294 115.1128 0)
@@
       (effects (font (size 1.27 1.27)) hide)
     )
-    (property "Datasheet" "https://media.digikey.com/pdf/Data%20Sheets/Lite-On%20PDFs/LTST-S220GKT.pdf" (id 3) (at 287.02 118.11 0)
+    (property "Datasheet" "~" (id 3) (at 287.02 118.11 0)
       (effects (font (size 1.27 1.27)) hide)
     )
@@
       (effects (font (size 1.524 1.524)))
     )
-    (property "Footprint" "Sapphire:EVQP7C01P" (id 2) (at 205.74 66.04 0)
+    (property "Footprint" "Sapphire:EVQP7C01P_HandSolder" (id 2) (at 205.74 66.04 0)
       (effects (font (size 1.524 1.524)))
     )
@@
     (pin "S1")
   )
+  (symbol (lib_id "power:PWR_FLAG") (at 97.79 61.468 90) (unit 1)
+    (in_bom yes) (on_board yes) (fields_autoplaced)
+    (property "Reference" "#FLG0106" (id 0) (at 95.885 61.468 0)
+      (effects (font (size 1.27 1.27)) hide)
+    )
+    (property "Value" "PWR_FLAG" (id 1) (at 94.6151 61.9018 90)
+      (effects (font (size 1.27 1.27)) (justify left))
+    )
+    (property "Footprint" "" (id 2) (at 97.79 61.468 0)
+      (effects (font (size 1.27 1.27)) hide)
+    )
+    (property "Datasheet" "~" (id 3) (at 97.79 61.468 0)
+      (effects (font (size 1.27 1.27)) hide)
+    )
+    (pin "1")
+  )
   (symbol (lib_id "Device:FerriteBead") (at 337.82 67.31 90) (unit 1)
