File: SapphireMini_SD.kicad_sch (KiCad schematic)
At the start: 13 parts, among them J301 503182-1852, U301 MB85RS2MTAPNF-G-BDERE1

Commit message: InProgress
Parts:
- gave numbers to parts that had none: 1
Changed lines of the file:
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@@
   (symbol (lib_id "Device:R_Small_US") (at 26.67 92.71 180) (unit 1)
     (in_bom yes) (on_board yes)
-    (property "Reference" "R?" (id 0) (at 29.21 90.17 0)
+    (property "Reference" "R302" (id 0) (at 29.21 90.17 0)
       (effects (font (size 1.27 1.27)) (justify left))
     )

Commit message: M2R2 basic DRC passed
Parts:
- U301: footprint Package_SO:SOP-8_3.9x4.9mm_P1.27mm -> Sapphire:SOP-8_3.9x4.9mm_P1.27mm
Changed lines of the file:
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@@
     (property "Reference" "U301" (id 0) (at 66.04 92.71 0))
     (property "Value" "MB85RS2MTAPNF-G-BDERE1" (id 1) (at 55.88 90.17 0))
-    (property "Footprint" "Package_SO:SOP-8_3.9x4.9mm_P1.27mm" (id 2) (at 54.61 100.33 0)
+    (property "Footprint" "Sapphire:SOP-8_3.9x4.9mm_P1.27mm" (id 2) (at 54.61 100.33 0)
       (effects (font (size 1.27 1.27)) hide)
     )

Commit message: Added slot for wiring
Parts:
- R301, R302: MPN CRCW060347R0FKEAC -> CRCW060310K0FKEAC
- R304, R309: Manufacturer (none) -> Vishay
Changed lines of the file:
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@@
       (effects (font (size 1.27 1.27)) hide)
     )
-    (property "MPN" "CRCW060347R0FKEAC" (id 6) (at 31.75 92.71 0)
+    (property "MPN" "CRCW060310K0FKEAC" (id 6) (at 31.75 92.71 0)
       (effects (font (size 1.27 1.27)) hide)
     )
@@
       (effects (font (size 1.27 1.27)) hide)
     )
-    (property "Description" "47 Ohms ±1% 0.1W, 1/10W Chip Resistor 0603" (id 13) (at 31.75 92.71 0)
+    (property "Description" "10K Ohms ±1% 0.1W, 1/10W Chip Resistor 0603" (id 13) (at 31.75 92.71 0)
       (effects (font (size 1.27 1.27)) hide)
     )
@@
       (effects (font (size 1.27 1.27)) hide)
     )
-    (property "MPN" "CRCW060347R0FKEAC" (id 6) (at 26.67 92.71 0)
+    (property "MPN" "CRCW060310K0FKEAC" (id 6) (at 26.67 92.71 0)
       (effects (font (size 1.27 1.27)) hide)
     )
@@
       (effects (font (size 1.27 1.27)) hide)
     )
-    (property "Description" "47 Ohms ±1% 0.1W, 1/10W Chip Resistor 0603" (id 13) (at 26.67 92.71 0)
+    (property "Description" "10K Ohms ±1% 0.1W, 1/10W Chip Resistor 0603" (id 13) (at 26.67 92.71 0)
       (effects (font (size 1.27 1.27)) hide)
     )
@@
     )
     (property "MPN" "CRCW060347R0FKEAC" (id 5) (at 80.01 101.6 0)
+      (effects (font (size 1.27 1.27)) hide)
+    )
+    (property "Manufacturer" "Vishay" (id 6) (at 80.01 101.6 0)
       (effects (font (size 1.27 1.27)) hide)
     )
@@
       (effects (font (size 1.27 1.27)) hide)
     )
+    (property "Manufacturer" "Vishay" (id 6) (at 223.52 99.06 0)
+      (effects (font (size 1.27 1.27)) hide)
+    )

Commit message: OSH_ParkM2R3
Parts:
- FB301, J301, R304, R309: Populate (none) -> 1
Changed lines of the file:
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@@
+      (effects (font (size 1.27 1.27)) hide)
+    )
+    (property "Populate" "1" (id 7) (at 80.01 101.6 0)
       (effects (font (size 1.27 1.27)) hide)
     )
@@
       (effects (font (size 1.27 1.27)) hide)
     )
+    (property "Populate" "1" (id 7) (at 223.52 99.06 0)
+      (effects (font (size 1.27 1.27)) hide)
+    )
     (pin "1")
     (pin "2")
@@
     )
     (property "Manufacturer" "Amphenol ICC (FCI)" (id 7) (at 245.11 99.06 0)
+      (effects (font (size 1.27 1.27)) hide)
+    )
+    (property "Populate" "1" (id 8) (at 245.11 99.06 0)
       (effects (font (size 1.27 1.27)) hide)
     )
@@
       (effects (font (size 1.27 1.27)) hide)
     )
+    (property "Populate" "1" (id 6) (at 157.48 96.52 0)
+      (effects (font (size 1.27 1.27)) hide)
+    )

Commit message: Board ready for final check
Changed lines of the file:
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@@
   (junction (at 184.15 96.52) (diameter 0) (color 0 0 0 0)
   )
+  (junction (at 168.9047 96.52) (diameter 0) (color 0 0 0 0)
+  )
   (wire (pts (xy 173.99 109.22) (xy 173.99 113.03))
     (stroke (width 0) (type default) (color 0 0 0 0))
@@
     (stroke (width 0) (type default) (color 0 0 0 0))
   )
+  (wire (pts (xy 168.9047 96.52) (xy 173.99 96.52))
+    (stroke (width 0) (type default) (color 0 0 0 0))
+  )
   (wire (pts (xy 227.33 86.36) (xy 226.06 85.09))
     (stroke (width 0) (type default) (color 0 0 0 0))
@@
     (stroke (width 0) (type default) (color 0 0 0 0))
   )
-  (wire (pts (xy 163.83 96.52) (xy 173.99 96.52))
+  (wire (pts (xy 163.83 96.52) (xy 168.9047 96.52))
     (stroke (width 0) (type default) (color 0 0 0 0))
   )
@@
       (effects (font (size 1.27 1.27)) hide)
     )
+    (pin "1")
+  )
+  (symbol (lib_id "power:PWR_FLAG") (at 168.9047 96.52 0) (unit 1)
+    (in_bom yes) (on_board yes) (fields_autoplaced)
+    (property "Reference" "#FLG0101" (id 0) (at 168.9047 94.615 0)
+      (effects (font (size 1.27 1.27)) hide)
+    )
+    (property "Value" "PWR_FLAG" (id 1) (at 168.9047 92.9442 0))
+    (property "Footprint" "" (id 2) (at 168.9047 96.52 0)
+      (effects (font (size 1.27 1.27)) hide)
+    )
+    (property "Datasheet" "~" (id 3) (at 168.9047 96.52 0)
+      (effects (font (size 1.27 1.27)) hide)
+    )
