File: SapphireMini_WIFI.kicad_sch (KiCad schematic)
At the start: 11 parts, among them M701 AdafruitWINC1500

Commit message: Midst of pretying layout
Parts:
- added R605: 47, Resistor_SMD:R_0603_1608Metric, symbol Device:R_US
Connections:
- net at M701.10 (WAKE): now also R605.1
- new net SPARE: R605.2
- no-connect marks 4 -> 3
Changed lines of the file:
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@@
   )
   (no_connect (at 165.1 96.52))
-  (no_connect (at 165.1 88.9))
   (no_connect (at 165.1 91.44))
   (no_connect (at 165.1 93.98))
@@
     (stroke (width 0) (type default) (color 0 0 0 0))
   )
+  (wire (pts (xy 134.62 88.9) (xy 152.4 88.9))
+    (stroke (width 0) (type default) (color 0 0 0 0))
+  )
   (wire (pts (xy 134.62 71.12) (xy 165.1 71.12))
     (stroke (width 0) (type default) (color 0 0 0 0))
@@
   )
   (wire (pts (xy 165.1 66.04) (xy 162.56 66.04))
+    (stroke (width 0) (type default) (color 0 0 0 0))
+  )
+  (wire (pts (xy 165.1 88.9) (xy 160.02 88.9))
     (stroke (width 0) (type default) (color 0 0 0 0))
   )
@@
   )
   (hierarchical_label "SPI_MISO" (shape output) (at 105.41 73.66 180)
+    (effects (font (size 1.27 1.27)) (justify right))
+  )
+  (hierarchical_label "SPARE" (shape input) (at 134.62 88.9 180)
     (effects (font (size 1.27 1.27)) (justify right))
   )
@@
       (effects (font (size 1.27 1.27)) hide)
     )
+    (pin "1")
+    (pin "2")
+  )
+  (symbol (lib_id "Device:R_US") (at 156.21 88.9 270) (unit 1)
+    (in_bom yes) (on_board yes)
+    (property "Reference" "R605" (id 0) (at 151.13 87.63 90))
+    (property "Value" "47" (id 1) (at 158.75 87.63 90))
+    (property "Footprint" "Resistor_SMD:R_0603_1608Metric" (id 2) (at 155.956 89.916 90)
+      (effects (font (size 1.27 1.27)) hide)
+    )
+    (property "Datasheet" "~" (id 3) (at 156.21 88.9 0)
+      (effects (font (size 1.27 1.27)) hide)
+    )
+    (property "Description" "47 Ohms ±1% 0.1W, 1/10W Chip Resistor 0603" (id 4) (at 156.21 88.9 0)
+      (effects (font (size 1.27 1.27)) hide)
+    )
+    (property "MPN" "CRCW060347R0FKEAC" (id 5) (at 156.21 88.9 0)
+      (effects (font (size 1.27 1.27)) hide)
+    )

Commit message: Added slot for wiring
Parts:
- R603, R604, R605, R702, R703: Manufacturer (none) -> Vishay
Changed lines of the file:
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@@
+      (effects (font (size 1.27 1.27)) hide)
+    )
+    (property "Manufacturer" "Vishay" (id 6) (at 114.3 66.04 0)
       (effects (font (size 1.27 1.27)) hide)
     )
@@
       (effects (font (size 1.27 1.27)) hide)
     )
+    (property "Manufacturer" "Vishay" (id 6) (at 156.21 88.9 0)
+      (effects (font (size 1.27 1.27)) hide)
+    )
     (pin "1")
     (pin "2")
@@
       (effects (font (size 1.27 1.27)) hide)
     )
+    (property "Manufacturer" "Vishay" (id 6) (at 113.03 78.74 0)
+      (effects (font (size 1.27 1.27)) hide)
+    )
     (pin "1")
     (pin "2")
@@
       (effects (font (size 1.27 1.27)) hide)
     )
+    (property "Manufacturer" "Vishay" (id 6) (at 114.3 68.58 0)
+      (effects (font (size 1.27 1.27)) hide)
+    )
     (pin "1")
     (pin "2")
@@
       (effects (font (size 1.27 1.27)) hide)
     )
+    (property "Manufacturer" "Vishay" (id 6) (at 113.03 76.2 0)
+      (effects (font (size 1.27 1.27)) hide)
+    )

Commit message: OSH_ParkM2R3
Parts:
- FB701, R603, R604, R605: Populate (none) -> 1
- M701: value AdafruitWINC1500 -> DNP AdafruitWINC1500; Populate (none) -> 0
- R602: value 0 -> DNP 0; Populate 1 -> 0
- R702, R703: value 47 -> DNP 47; Populate (none) -> 0
Changed lines of the file:
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@@
       (effects (font (size 1.27 1.27)) (justify left))
     )
-    (property "Value" "AdafruitWINC1500" (id 1) (at 183.5912 81.788 0)
+    (property "Value" "DNP AdafruitWINC1500" (id 1) (at 183.5912 81.788 0)
       (effects (font (size 1.27 1.27)) (justify left))
     )
@@
     )
     (property "Description" "Adafruit Winc1500 breakout" (id 4) (at 170.18 66.04 0)
+      (effects (font (size 1.27 1.27)) hide)
+    )
+    (property "Populate" "0" (id 5) (at 170.18 66.04 0)
       (effects (font (size 1.27 1.27)) hide)
     )
@@
       (effects (font (size 1.27 1.27)) hide)
     )
+    (property "Populate" "1" (id 7) (at 114.3 66.04 0)
+      (effects (font (size 1.27 1.27)) hide)
+    )
     (pin "1")
     (pin "2")
@@
       (effects (font (size 1.27 1.27)) hide)
     )
+    (property "Populate" "1" (id 7) (at 156.21 88.9 0)
+      (effects (font (size 1.27 1.27)) hide)
+    )
     (pin "1")
     (pin "2")
@@
     (in_bom yes) (on_board yes)
     (property "Reference" "R703" (id 0) (at 109.22 77.47 90))
-    (property "Value" "47" (id 1) (at 115.57 77.47 90))
+    (property "Value" "DNP 47" (id 1) (at 115.57 77.47 90))
     (property "Footprint" "Resistor_SMD:R_0603_1608Metric" (id 2) (at 112.776 79.756 90)
       (effects (font (size 1.27 1.27)) hide)
@@
       (effects (font (size 1.27 1.27)) hide)
     )
+    (property "Populate" "0" (id 7) (at 113.03 78.74 0)
+      (effects (font (size 1.27 1.27)) hide)
+    )
     (pin "1")
     (pin "2")
@@
     (in_bom yes) (on_board yes)
     (property "Reference" "R702" (id 0) (at 110.49 67.31 90))
-    (property "Value" "47" (id 1) (at 116.84 67.31 90))
+    (property "Value" "DNP 47" (id 1) (at 116.84 67.31 90))
     (property "Footprint" "Resistor_SMD:R_0603_1608Metric" (id 2) (at 114.046 69.596 90)
       (effects (font (size 1.27 1.27)) hide)
@@
     )
     (property "Manufacturer" "Vishay" (id 6) (at 114.3 68.58 0)
+      (effects (font (size 1.27 1.27)) hide)
+    )
+    (property "Populate" "0" (id 7) (at 114.3 68.58 0)
       (effects (font (size 1.27 1.27)) hide)
     )
@@
       (effects (font (size 1.27 1.27)) (justify right))
     )
-    (property "Value" "0" (id 1) (at 115.57 72.39 90)
+    (property "Value" "DNP 0" (id 1) (at 115.57 72.39 90)
       (effects (font (size 1.27 1.27)) (justify right))
     )
@@
       (effects (font (size 1.27 1.27)) hide)
     )
-    (property "Populate" "1" (id 7) (at 113.03 73.66 0)
+    (property "Populate" "0" (id 7) (at 113.03 73.66 0)
       (effects (font (size 1.27 1.27)) hide)
     )
@@
     )
     (property "Manufacturer" "Vishay" (id 6) (at 113.03 76.2 0)
+      (effects (font (size 1.27 1.27)) hide)
+    )
+    (property "Populate" "1" (id 7) (at 113.03 76.2 0)
       (effects (font (size 1.27 1.27)) hide)
     )
@@
       (effects (font (size 1.27 1.27)) hide)
     )
+    (property "Populate" "1" (id 6) (at 132.08 45.72 0)
+      (effects (font (size 1.27 1.27)) hide)
+    )

Commit message: Board ready for final check
Parts:
- R602, R702, R703: now left out of the parts list
- R605: value 47 -> DNP 47; now left out of the parts list
Changed lines of the file:
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@@
   (junction (at 120.65 68.58) (diameter 0) (color 0 0 0 0)
+  )
+  (junction (at 141.732 45.72) (diameter 0) (color 0 0 0 0)
   )
   (junction (at 149.86 53.34) (diameter 0) (color 0 0 0 0)
@@
     (stroke (width 0) (type default) (color 0 0 0 0))
   )
-  (wire (pts (xy 138.43 45.72) (xy 149.86 45.72))
+  (wire (pts (xy 138.43 45.72) (xy 141.732 45.72))
     (stroke (width 0) (type default) (color 0 0 0 0))
   )
@@
   )
   (wire (pts (xy 132.08 68.58) (xy 134.62 71.12))
+    (stroke (width 0) (type default) (color 0 0 0 0))
+  )
+  (wire (pts (xy 141.732 45.72) (xy 149.86 45.72))
     (stroke (width 0) (type default) (color 0 0 0 0))
   )
@@
     (pin "2")
   )
+  (symbol (lib_id "power:PWR_FLAG") (at 141.732 45.72 0) (unit 1)
+    (in_bom yes) (on_board yes) (fields_autoplaced)
+    (property "Reference" "#FLG0105" (id 0) (at 141.732 43.815 0)
+      (effects (font (size 1.27 1.27)) hide)
+    )
+    (property "Value" "PWR_FLAG" (id 1) (at 141.732 42.1442 0))
+    (property "Footprint" "" (id 2) (at 141.732 45.72 0)
+      (effects (font (size 1.27 1.27)) hide)
+    )
+    (property "Datasheet" "~" (id 3) (at 141.732 45.72 0)
+      (effects (font (size 1.27 1.27)) hide)
+    )
+    (pin "1")
+  )
   (symbol (lib_id "Device:R_US") (at 156.21 88.9 270) (unit 1)
-    (in_bom yes) (on_board yes)
+    (in_bom no) (on_board yes)
     (property "Reference" "R605" (id 0) (at 151.13 87.63 90))
-    (property "Value" "47" (id 1) (at 158.75 87.63 90))
+    (property "Value" "DNP 47" (id 1) (at 158.75 87.63 90))
     (property "Footprint" "Resistor_SMD:R_0603_1608Metric" (id 2) (at 155.956 89.916 90)
       (effects (font (size 1.27 1.27)) hide)
@@
   )
   (symbol (lib_id "Device:R_US") (at 113.03 78.74 270) (unit 1)
-    (in_bom yes) (on_board yes)
+    (in_bom no) (on_board yes)
     (property "Reference" "R703" (id 0) (at 109.22 77.47 90))
     (property "Value" "DNP 47" (id 1) (at 115.57 77.47 90))
@@
   )
   (symbol (lib_id "Device:R_US") (at 114.3 68.58 270) (unit 1)
-    (in_bom yes) (on_board yes)
+    (in_bom no) (on_board yes)
     (property "Reference" "R702" (id 0) (at 110.49 67.31 90))
     (property "Value" "DNP 47" (id 1) (at 116.84 67.31 90))
@@
   )
   (symbol (lib_id "Device:R_Small_US") (at 113.03 73.66 90) (unit 1)
-    (in_bom yes) (on_board yes)
+    (in_bom no) (on_board yes)
     (property "Reference" "R602" (id 0) (at 107.95 72.39 90)
       (effects (font (size 1.27 1.27)) (justify right))
